File: Connectors.kicad_sch (KiCad schematic)
At the start: 4 parts, among them J1 Conn_01x04_Pin, J2 Conn_01x04_Pin, J3 Conn_01x09_Pin, J4 Conn_02x03_Odd_Even

Commit message: Begun giving values to components
Parts:
- renumbered J4 to J?, J2 to J?, J1 to J?, J3 to J?
Changed lines of the file:
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@@
   (symbol (lib_id "Connector_Generic:Conn_02x03_Odd_Even") (at 195.58 143.51 0) (unit 1)
     (in_bom yes) (on_board yes) (dnp no)
-    (property "Reference" "J4" (at 196.85 134.62 0)
+    (property "Reference" "J?" (at 196.85 134.62 0)
       (effects (font (size 1.27 1.27)))
     )
@@
       (project "MCUDatalogger"
         (path "/a46afdbf-01b2-4464-8083-80e47ae67da1/803d4b1a-ac34-47b6-b579-d41bb776d097"
-          (reference "J4") (unit 1)
+          (reference "J?") (unit 1)
         )
       )
@@
   (symbol (lib_id "Connector:Conn_01x04_Pin") (at 191.77 118.11 0) (unit 1)
     (in_bom yes) (on_board yes) (dnp no)
-    (property "Reference" "J2" (at 192.405 110.49 0)
+    (property "Reference" "J?" (at 192.405 110.49 0)
       (effects (font (size 1.27 1.27)))
     )
@@
       (project "MCUDatalogger"
         (path "/a46afdbf-01b2-4464-8083-80e47ae67da1/803d4b1a-ac34-47b6-b579-d41bb776d097"
-          (reference "J2") (unit 1)
+          (reference "J?") (unit 1)
         )
       )
@@
   (symbol (lib_id "Connector:Conn_01x04_Pin") (at 173.99 118.11 0) (unit 1)
     (in_bom yes) (on_board yes) (dnp no)
-    (property "Reference" "J1" (at 174.625 110.49 0)
+    (property "Reference" "J?" (at 174.625 110.49 0)
       (effects (font (size 1.27 1.27)))
     )
@@
       (project "MCUDatalogger"
         (path "/a46afdbf-01b2-4464-8083-80e47ae67da1/803d4b1a-ac34-47b6-b579-d41bb776d097"
-          (reference "J1") (unit 1)
+          (reference "J?") (unit 1)
         )
       )
@@
   (symbol (lib_id "Connector:Conn_01x09_Pin") (at 173.99 146.05 0) (unit 1)
     (in_bom yes) (on_board yes) (dnp no)
-    (property "Reference" "J3" (at 174.625 130.81 0)
+    (property "Reference" "J?" (at 174.625 130.81 0)
       (effects (font (size 1.27 1.27)))
     )
@@
       (project "MCUDatalogger"
         (path "/a46afdbf-01b2-4464-8083-80e47ae67da1/803d4b1a-ac34-47b6-b579-d41bb776d097"
-          (reference "J3") (unit 1)
+          (reference "J?") (unit 1)
         )
       )
