File: MCUDatalogger.kicad_sch (KiCad schematic)
At the start: 25 parts, among them U1 24LC1025, U2 24LC1025, U3 DS1337S_, U4 ATMEGA328P-AU, Y1 Crystal, Y2 Crystal

Commit message: Begun giving values to components
Parts:
- R1: renamed from R4; value R -> 10K
- Y1: value Crystal -> 32.768 KHz
- renumbered BT1 to BT?, C5 to C?, C1 to C?, C4 to C?, C3 to C?, C2 to C?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
